File: quartet_main.sch (KiCad schematic (older format))
At the start: 18 parts, among them J1 USB_C_Receptacle_USB2.0, J2 AVR-ISP-6, J3 Conn_01x16, J4 Conn_01x04

Commit message: Move board connectors to separate sheets, create breakout board for testing halves
Parts:
- removed J3: Conn_01x16, Gigahawk:F519-1A7A1-11016-E200, symbol Connector_Generic:Conn_01x16
- removed J4: Conn_01x04, Gigahawk:F519-1A7A1-11004-E200, symbol Connector_Generic:Conn_01x04
Connections:
- wire segments 120 -> 96
Changed lines of the file:
@@
 $Descr A4 11693 8268
 encoding utf-8
-Sheet 2 2
+Sheet 2 3
 Title ""
 Date ""
@@
 	3100 2100 3000 2100
 $Comp
-L power:+5V #PWR016
-U 1 1 60058F3A
-P 9800 1350
-F 0 "#PWR016" H 9800 1200 50  0001 C CNN
-F 1 "+5V" H 9815 1523 50  0000 C CNN
-F 2 "" H 9800 1350 50  0001 C CNN
-F 3 "" H 9800 1350 50  0001 C CNN
-	1    9800 1350
-	1    0    0    -1
-$EndComp
-$Comp
-L power:GND #PWR017
-U 1 1 600597C0
-P 9800 1850
-F 0 "#PWR017" H 9800 1600 50  0001 C CNN
-F 1 "GND" H 9805 1677 50  0000 C CNN
-F 2 "" H 9800 1850 50  0001 C CNN
-F 3 "" H 9800 1850 50  0001 C CNN
-	1    9800 1850
-	1    0    0    -1
-$EndComp
-Wire Wire Line
-	9900 1450 9800 1450
-Wire Wire Line
-	9800 1450 9800 1350
-Wire Wire Line
-	9900 1550 9800 1550
-Wire Wire Line
-	9800 1550 9800 1450
-Connection ~ 9800 1450
-Wire Wire Line
-	9900 1750 9800 1750
-Wire Wire Line
-	9800 1750 9800 1850
-Wire Wire Line
-	9900 1650 9800 1650
-Wire Wire Line
-	9800 1650 9800 1750
-Connection ~ 9800 1750
-Text GLabel 8800 1550 0    50   Input ~ 0
-PD1
-Text GLabel 8800 1450 0    50   Input ~ 0
-PD0
-Text GLabel 8800 1650 0    50   Input ~ 0
-PD5
-Text GLabel 8800 1750 0    50   Input ~ 0
-PD6
-Text GLabel 8800 1850 0    50   Input ~ 0
-PD7
-Text GLabel 8800 1950 0    50   Input ~ 0
-PB0
-Text GLabel 8800 2050 0    50   Input ~ 0
-PB1
-Text GLabel 8800 2150 0    50   Input ~ 0
-PB2
-Text GLabel 8800 2250 0    50   Input ~ 0
-PC2
-Text GLabel 8800 2350 0    50   Input ~ 0
-PC3
-Text GLabel 8800 2450 0    50   Input ~ 0
-ADC7
-Wire Wire Line
-	8800 2450 8900 2450
-Wire Wire Line
-	8900 2350 8800 2350
-Wire Wire Line
-	8800 2250 8900 2250
-Wire Wire Line
-	8900 2150 8800 2150
-Wire Wire Line
-	8800 2050 8900 2050
-Wire Wire Line
-	8900 1950 8800 1950
-Wire Wire Line
-	8800 1850 8900 1850
-Wire Wire Line
-	8900 1750 8800 1750
-Wire Wire Line
-	8800 1650 8900 1650
-Wire Wire Line
-	8900 1550 8800 1550
-Wire Wire Line
-	8800 1450 8900 1450
-$Comp
-L Connector_Generic:Conn_01x16 J3
-U 1 1 600CBF49
-P 9100 2150
-F 0 "J3" H 9180 2142 50  0000 L CNN
-F 1 "Conn_01x16" H 9180 2051 50  0000 L CNN
-F 2 "Gigahawk:F519-1A7A1-11016-E200" H 9100 2150 50  0001 C CNN
-F 3 "~" H 9100 2150 50  0001 C CNN
-	1    9100 2150
-	1    0    0    -1
-$EndComp
-$Comp
-L Connector_Generic:Conn_01x04 J4
-U 1 1 600D0AD0
-P 10100 1550
-F 0 "J4" H 10180 1542 50  0000 L CNN
-F 1 "Conn_01x04" H 10180 1451 50  0000 L CNN
-F 2 "Gigahawk:F519-1A7A1-11004-E200" H 10100 1550 50  0001 C CNN
-F 3 "~" H 10100 1550 50  0001 C CNN
-	1    10100 1550
-	1    0    0    -1
-$EndComp
-Text GLabel 8800 2650 0    50   Input ~ 0
-MISO
-Text GLabel 8800 2750 0    50   Input ~ 0
-MOSI
-Text GLabel 8800 2550 0    50   Input ~ 0
-SCK
-Text GLabel 8800 2950 0    50   Input ~ 0
-SDA
-Text GLabel 8800 2850 0    50   Input ~ 0
-SCL
-Wire Wire Line
-	8800 2550 8900 2550
-Wire Wire Line
-	8800 2650 8900 2650
-Wire Wire Line
-	8800 2750 8900 2750
-Wire Wire Line
-	8800 2850 8900 2850
-Wire Wire Line
-	8800 2950 8900 2950
-$Comp
 L Device:R R7
 U 1 1 601191CE
@@
 Wire Wire Line
 	4200 1500 4200 1400
+$Sheet
+S 8050 1400 1150 350
+U 5FF7CBCC
+F0 "reciever_main" 50
+F1 "reciever_main.sch" 50
+$EndSheet
 $EndSCHEMATC

Commit message: Reroute matrix, redo schematics for feather compat
Parts:
- removed A1: ARDUINO_PRO_MINI, Gigahawk:ARDUINO_PRO_MINI_THT, symbol gigahawk:ARDUINO_PRO_MINI
- removed A3: POWERBOOST_1000C, Gigahawk:POWERBOOST_1000C_THT, symbol gigahawk:POWERBOOST_1000C
- removed D1, D2: 3.6V, Diode_SMD:D_SOT-23_ANK, symbol Device:D_Zener
- removed J1: USB_C_Receptacle_USB2.0, Gigahawk:USB_C_Receptacle_GCT_USB4085, symbol Connector:USB_C_Receptacle_USB2.0
- removed J2: AVR-ISP-6, Gigahawk:AVR-ISP-6, symbol Connector:AVR-ISP-6
- removed R3: 1.5k, Resistor_SMD:R_0805_2012Metric_Pad1.15x1.40mm_HandSolder, symbol Device:R
- removed R4: DNI, Resistor_SMD:R_0805_2012Metric_Pad1.15x1.40mm_HandSolder, symbol Device:R
- removed R5, R6: 22R, Resistor_SMD:R_0805_2012Metric_Pad1.15x1.40mm_HandSolder, symbol Device:R
- removed S1: EG2219, Gigahawk:SW_EG2219, symbol gigahawk:EG2219
- added A1: Adafruit_Feather_Generic, Gigahawk:Adafruit_Feather_LowProfileSocket, symbol gigahawk:Adafruit_Feather_Generic
- added SW1: SW_SPDT, Button_Switch_THT:SW_E-Switch_EG1224_SPDT_Angled, symbol Switch:SW_SPDT
- added SW?: SW_Push, symbol Switch:SW_Push
- added TP? (x3): TestPoint, symbol Connector:TestPoint
- R1, R2: value 5.1k -> 100k
Connections:
- net labels added: +3V3, +BATT, A0, A1, A2, A3, A4, A5, D0, D1, D2, D3, EN, RX_MCU, SPARE, TX_MCU, ~RESET
- net labels removed: +5V, ADC7, BOOST_EN, BOOST_LBO, BOOST_OUT, BOOST_VS, PB0, PB1, PB2, PC2, PC3, PD0, PD1, PD5, PD6, PD7, RST, USB_D+, USB_D-, VBAT, VUSB
- wire segments 96 -> 57
- no-connect marks 7 -> 3
Other:
- note added: "Disconnect EN from \nground to enable 3V3\n"
- note added: "External battery divider for boards \nthat don't have an internal one"
- note added: "USB power may only be available \nwhen USB is actually connected"
- note removed: "Connect BOOST_EN to GND to\ndisable PowerBoost Module\n"
- moved on the sheet: A2

Commit message: Finish and route quartet mainboard
Parts:
- added TP4: TestPoint, TestPoint:TestPoint_Pad_1.0x1.0mm, symbol Connector:TestPoint
- SW2: renamed from SW?; footprint (none) -> Button_Switch_SMD:SW_SPST_TL3342
- TP1, TP2, TP3: renamed from TP?; footprint (none) -> TestPoint:TestPoint_Pad_1.0x1.0mm
Connections:
- net BLE_CS: now also A1.25 (D6); no longer A1.23 (D4)
- net BLE_RST: now also A1.23 (D4); no longer A1.25 (D6)
- net GND: now also TP4.1
Other:
- moved on the sheet: TP2
Changed lines of the file:
@@
 $Descr A4 11693 8268
 encoding utf-8
-Sheet 2 3
+Sheet 2 4
 Title ""
 Date ""
@@
 	1300 2700 1400 2700
 $Comp
-L power:+3V3 #PWR?
+L power:+3V3 #PWR0101
 U 1 1 60438936
 P 7300 3950
-F 0 "#PWR?" H 7300 3800 50  0001 C CNN
+F 0 "#PWR0101" H 7300 3800 50  0001 C CNN
 F 1 "+3V3" H 7315 4123 50  0000 C CNN
 F 2 "" H 7300 3950 50  0001 C CNN
@@
 NoConn ~ 2400 1700
 $Comp
-L Switch:SW_Push SW?
+L Switch:SW_Push SW2
 U 1 1 6043A24B
 P 3450 6800
-F 0 "SW?" H 3450 7085 50  0000 C CNN
+F 0 "SW2" H 3450 7085 50  0000 C CNN
 F 1 "SW_Push" H 3450 6994 50  0000 C CNN
-F 2 "" H 3450 7000 50  0001 C CNN
+F 2 "Button_Switch_SMD:SW_SPST_TL3342" H 3450 7000 50  0001 C CNN
 F 3 "~" H 3450 7000 50  0001 C CNN
 	1    3450 6800
@@
 	3250 6800 3150 6800
 $Comp
-L power:GND #PWR?
+L power:GND #PWR0102
 U 1 1 6043B659
 P 3750 6900
-F 0 "#PWR?" H 3750 6650 50  0001 C CNN
+F 0 "#PWR0102" H 3750 6650 50  0001 C CNN
 F 1 "GND" H 3755 6727 50  0000 C CNN
 F 2 "" H 3750 6900 50  0001 C CNN
@@
 Wire Wire Line
 	2400 2400 2500 2400
-Text GLabel 1300 1700 0    50   Input ~ 0
+Text GLabel 1300 1900 0    50   Input ~ 0
 BLE_CS
 Text GLabel 1300 1800 0    50   Input ~ 0
 BLE_IRQ
-Text GLabel 1300 1900 0    50   Input ~ 0
+Text GLabel 1300 1700 0    50   Input ~ 0
 BLE_RST
 Wire Wire Line
@@
 	1300 1900 1400 1900
 $Comp
-L Connector:TestPoint TP?
+L Connector:TestPoint TP2
 U 1 1 6045D861
-P 4300 7150
-F 0 "TP?" H 4242 7176 50  0000 R CNN
-F 1 "TestPoint" H 4242 7267 50  0000 R CNN
-F 2 "" H 4500 7150 50  0001 C CNN
-F 3 "~" H 4500 7150 50  0001 C CNN
-	1    4300 7150
+P 4300 7200
+F 0 "TP2" H 4242 7226 50  0000 R CNN
+F 1 "TestPoint" H 4242 7317 50  0000 R CNN
+F 2 "TestPoint:TestPoint_Pad_1.0x1.0mm" H 4500 7200 50  0001 C CNN
+F 3 "~" H 4500 7200 50  0001 C CNN
+	1    4300 7200
 	-1   0    0    1
 $EndComp
@@
 BLE_DFU
 $Comp
-L Connector:TestPoint TP?
+L Connector:TestPoint TP1
 U 1 1 6046442D
 P 4300 6700
-F 0 "TP?" H 4242 6726 50  0000 R CNN
+F 0 "TP1" H 4242 6726 50  0000 R CNN
 F 1 "TestPoint" H 4242 6817 50  0000 R CNN
-F 2 "" H 4500 6700 50  0001 C CNN
+F 2 "TestPoint:TestPoint_Pad_1.0x1.0mm" H 4500 6700 50  0001 C CNN
 F 3 "~" H 4500 6700 50  0001 C CNN
 	1    4300 6700
@@
 $EndComp
 $Comp
-L power:+BATT #PWR?
+L power:+BATT #PWR0103
 U 1 1 6046551C
 P 4300 6600
-F 0 "#PWR?" H 4300 6450 50  0001 C CNN
+F 0 "#PWR0103" H 4300 6450 50  0001 C CNN
 F 1 "+BATT" H 4315 6773 50  0000 C CNN
 F 2 "" H 4300 6600 50  0001 C CNN
@@
 	4300 6600 4300 6700
 $Comp
-L power:+3V3 #PWR?
+L power:+3V3 #PWR0104
 U 1 1 60466F30
 P 4800 6600
-F 0 "#PWR?" H 4800 6450 50  0001 C CNN
+F 0 "#PWR0104" H 4800 6450 50  0001 C CNN
 F 1 "+3V3" H 4815 6773 50  0000 C CNN
 F 2 "" H 4800 6600 50  0001 C CNN
@@
 $EndComp
 $Comp
-L Connector:TestPoint TP?
+L Connector:TestPoint TP3
 U 1 1 6046764D
 P 4800 6700
-F 0 "TP?" H 4742 6726 50  0000 R CNN
+F 0 "TP3" H 4742 6726 50  0000 R CNN
 F 1 "TestPoint" H 4742 6817 50  0000 R CNN
-F 2 "" H 5000 6700 50  0001 C CNN
+F 2 "TestPoint:TestPoint_Pad_1.0x1.0mm" H 5000 6700 50  0001 C CNN
 F 3 "~" H 5000 6700 50  0001 C CNN
 	1    4800 6700
@@
 Wire Wire Line
 	4800 6700 4800 6600
-Text GLabel 4300 7050 2    50   Input ~ 0
+Text GLabel 4300 7100 2    50   Input ~ 0
 BLE_DFU
 Wire Wire Line
-	4300 7150 4300 7050
+	4300 7200 4300 7100
 Wire Wire Line
 	7300 4650 7200 4650
+$Comp
+L power:GND #PWR0106
+U 1 1 6055FA3C
+P 4800 7100
+F 0 "#PWR0106" H 4800 6850 50  0001 C CNN
+F 1 "GND" H 4805 6927 50  0000 C CNN
+F 2 "" H 4800 7100 50  0001 C CNN
+F 3 "" H 4800 7100 50  0001 C CNN
+	1    4800 7100
+	-1   0    0    1
+$EndComp
+$Comp
+L Connector:TestPoint TP4
+U 1 1 60561683
+P 4800 7200
+F 0 "TP4" H 4742 7226 50  0000 R CNN
+F 1 "TestPoint" H 4742 7317 50  0000 R CNN
+F 2 "TestPoint:TestPoint_Pad_1.0x1.0mm" H 5000 7200 50  0001 C CNN
+F 3 "~" H 5000 7200 50  0001 C CNN
+	1    4800 7200
+	-1   0    0    1
+$EndComp
+Wire Wire Line
+	4800 7200 4800 7100
 $EndSCHEMATC
